Commit message: New yaml configs; New go urdf model

File: helios16p_ws/src/helios16p_cane_robot/urdf/helios16p.urdfverocondoggo.xacro (robot description, xacro)
@@ -8,13 +8,12 @@
   Licenza: GNU GPL
   -->
-  <!-- Global Shifts -->
   <xacro:property name="global_z_offset" value="0"/>
-  <xacro:property name="goshift_x" value="0.06"/>
-  <!-- Colors -->
+  <xacro:property name="goshift_x" value="0.09"/>
+  <!-- Colori -->
   <xacro:property name="waterblue" value="0 1 0.5 1"/>
   <xacro:property name="purple" value="1 0 1 1"/>
   <xacro:property name="gray" value="0.5 0.5 0.5 1"/>
   <xacro:property name="orange" value="1 0.5 0 0.5"/>
-  <!-- Sizes -->
+  <!-- Dimensioni ricorrenti -->
   <xacro:property name="base_box_size" value="0.065 0.12 0.05"/>
   <xacro:property name="top_box_size" value="0.065 0.12 0.01"/>
@@ -27,13 +26,10 @@
   <xacro:property name="lidar_radius" value="0.05"/>
   <xacro:property name="lidar_length" value="0.1"/>
-  <xacro:property name="gobody_fourth_of_y" value="0.06"/>
-  <xacro:property name="gobody_length" value="0.35"/>
-  <xacro:property name="halfpi" value="1.5708"/>
-  <!-- Positions -->
+  <!-- Posizioni ricorrenti -->
   <xacro:property name="base_round_z" value="0.025"/>
   <xacro:property name="top_z" value="0.145"/>
   <xacro:property name="pillar_z" value="0.05"/>
   <xacro:property name="lidar_z" value="0.05"/>
-  <!-- Base Link Its the "squared" part of the lidar base -->
+  <!-- Link principale - è la parte "squadrata" della base del lidar -->
   <link name="base_link">
     <visual>
@@ -47,5 +43,5 @@
     </visual>
   </link>
-<!-- Curved inferior part mounted on the main link -->
+<!-- parte curva inferiore montata sul link principale-->
   <link name="base_round_part">
     <visual>
@@ -64,5 +60,5 @@
     <origin xyz="0 0 ${base_round_z+global_z_offset}" rpy="0 0 0"/>
   </joint>
-<!-- Squared upper part mounted on the main link -->
+<!-- parte non curva superiore montata sul link principale-->
   <link name="top_link">
     <visual>
@@ -81,5 +77,5 @@
     <origin xyz="0 0 ${top_z+global_z_offset}" rpy="0 0 0"/>
   </joint>
-<!-- Curved upper part mounted on the main link -->
+<!-- parte curva superiore montata sul link principale-->
 <link name="top_round_part">
     <visual>
@@ -98,5 +94,5 @@
     <origin xyz="0 0 ${top_z+global_z_offset}" rpy="0 0 0"/>
   </joint>
-  <!-- Pillar mounted on the left side -->
+  <!-- Pilastro montato sul lato sinistro -->
   <link name="sx_pillar">
     <visual>
@@ -115,5 +111,5 @@
     <origin xyz="-0.055 0.05 ${pillar_z+global_z_offset}" rpy="0 0 0"/>
   </joint>
-  <!-- Pillar mounted on the right side -->
+  <!-- Pilastro montato sul lato destro -->
   <link name="dx_pillar">
     <visual>
@@ -132,5 +128,5 @@
     <origin xyz="-0.055 -0.05 ${pillar_z+global_z_offset}" rpy="0 0 0"/>
   </joint>
-  <!-- Lidar mounted on the base -->
+  <!-- Lidar montato sulla base -->
  <link name="lidar_link">
     <visual>
@@ -149,9 +145,8 @@
     <origin xyz="0 0 ${lidar_z+global_z_offset}" rpy="0 0 0"/>
   </joint>
-  <!-- Robot body parts -->
   <link name="gobody">
     <visual>
       <geometry>
-        <box size="${gobody_length} ${2 * gobody_fourth_of_y} ${2 * gobody_fourth_of_y}"/>
+        <box size="0.30 0.12 0.12"/>
       </geometry>
       <material name="gray">
@@ -164,10 +159,10 @@
     <parent link="base_link"/>
     <child link="gobody"/>
-    <origin xyz="${0-goshift_x} 0 ${-gobody_fourth_of_y+global_z_offset}" rpy="0 0 0"/>
+    <origin xyz="${0-goshift_x} 0 ${-0.06+global_z_offset}" rpy="0 0 0"/>
   </joint>
   <link name="gobodysx">
     <visual>
       <geometry>
-        <cylinder radius="${gobody_fourth_of_y}" length="${gobody_length}"/>
+        <cylinder radius="0.060" length="0.30"/>
       </geometry>
       <material name="gray">
@@ -180,10 +175,10 @@
     <parent link="base_link"/>
     <child link="gobodysx"/>
-    <origin xyz="${0-goshift_x} ${gobody_fourth_of_y} ${-gobody_fourth_of_y+global_z_offset}" rpy="0 ${halfpi} 0"/>
+    <origin xyz="${0-goshift_x} 0.06 ${-0.060+global_z_offset}" rpy="0 1.5708 0"/>
   </joint>
   <link name="gobodydx">
     <visual>
       <geometry>
-        <cylinder radius="${gobody_fourth_of_y}" length="${gobody_length}"/>
+        <cylinder radius="0.06" length="0.30"/>
       </geometry>
       <material name="gray">
@@ -196,11 +191,10 @@
     <parent link="base_link"/>
     <child link="gobodydx"/>
-    <origin xyz="${0-goshift_x} ${-gobody_fourth_of_y} ${-gobody_fourth_of_y+global_z_offset}" rpy="0 ${halfpi} 0"/>
-  </joint>
-  <!-- Neck -->
+    <origin xyz="${0-goshift_x} -0.06 ${-0.060+global_z_offset}" rpy="0 1.5708 0"/>
+  </joint>
   <link name="goneck">
     <visual>
       <geometry>
-        <box size="${gobody_fourth_of_y * 2} ${gobody_fourth_of_y} ${gobody_fourth_of_y * 2}"/>
+        <box size="0.15 0.08 0.12"/>
       </geometry>
       <material name="gray">
@@ -213,11 +207,10 @@
     <parent link="base_link"/>
     <child link="goneck"/>
-    <origin xyz="${(gobody_length / 2) + (gobody_fourth_of_y / 2) -goshift_x} 0 ${-gobody_fourth_of_y+global_z_offset}" rpy="0 0 0"/>
-  </joint>
-  <!-- Head -->
+    <origin xyz="${0.225-goshift_x} 0 ${-0.06+global_z_offset}" rpy="0 0 0"/>
+  </joint>
   <link name="gohead">
     <visual>
       <geometry>
-        <sphere radius="${gobody_fourth_of_y * 6 / 5}"/>
+        <sphere radius="0.072"/>
       </geometry>
       <material name="gray">
@@ -230,11 +223,106 @@
     <parent link="base_link"/>
     <child link="gohead"/>
-    <origin xyz="${(gobody_length / 2) + (gobody_fourth_of_y * 2) - goshift_x} 0 ${-gobody_fourth_of_y+global_z_offset}" rpy="${halfpi} 0 0"/>
-  </joint>
-  <!-- Back -->
-  <link name="goback">
-    <visual>
-      <geometry>
-        <cylinder radius="${gobody_fourth_of_y}" length="${gobody_fourth_of_y * 4}"/>
+    <origin xyz="${0.30-goshift_x} 0 ${-0.060+global_z_offset}" rpy="1.5708 0 0"/>
+  </joint>
+  <link name="goassback">
+    <visual>
+      <geometry>
+        <cylinder radius="0.06" length="0.18"/>
+      </geometry>
+      <material name="gray">
+        <color rgba="${gray}"/>
+      </material>
+      <origin xyz="0 0 0" rpy="0 0 0"/>
+    </visual>
+  </link>
+  <joint name="goassback_to_base" type="fixed">
+    <parent link="base_link"/>
+    <child link="goassback"/>
+    <origin xyz="${-0.15-goshift_x} 0 ${-0.060+global_z_offset}" rpy="1.5708 0 0"/>
+  </joint>
+  <link name="goassdx">
+    <visual>
+      <geometry>
+        <sphere radius="0.06"/>
+      </geometry>
+      <material name="gray">
+        <color rgba="${gray}"/>
+      </material>
+      <origin xyz="0 0 0" rpy="0 0 0"/>
+    </visual>
+  </link>
+  <joint name="goassdx_to_base" type="fixed">
+    <parent link="base_link"/>
+    <child link="goassdx"/>
+    <origin xyz="${-0.15-goshift_x} -0.09 ${-0.060+global_z_offset}" rpy="1.5708 0 0"/>
+  </joint>
+  <link name="goassx">
+    <visual>
+      <geometry>
+        <sphere radius="0.06"/>
+      </geometry>
+      <material name="gray">
+        <color rgba="${gray}"/>
+      </material>
+      <origin xyz="0 0 0" rpy="0 0 0"/>
+    </visual>
+  </link>
+  <joint name="goasssx_to_base" type="fixed">
+    <parent link="base_link"/>
+    <child link="goassx"/>
+    <origin xyz="${-0.15-goshift_x} 0.09 ${-0.060+global_z_offset}" rpy="1.5708 0 0"/>
+  </joint>
+<link name="goneckdx">
+    <visual>
+      <geometry>
+        <sphere radius="0.06"/>
+      </geometry>
+      <material name="gray">
+        <color rgba="${gray}"/>
+      </material>
+      <origin xyz="0 0 0" rpy="0 0 0"/>
+    </visual>
+  </link>
+  <joint name="goneckdx_to_base" type="fixed">
+    <parent link="base_link"/>
+    <child link="goneckdx"/>
+    <origin xyz="${0.15-goshift_x} -0.09 ${-0.060+global_z_offset}" rpy="1.5708 0 0"/>
+  </joint>
+  <link name="gonecksx">
+    <visual>
+      <geometry>
+        <sphere radius="0.06"/>
+      </geometry>
+      <material name="gray">
+        <color rgba="${gray}"/>
+      </material>
+      <origin xyz="0 0 0" rpy="0 0 0"/>
+    </visual>
+  </link>
+  <joint name="gonecksx_to_base" type="fixed">
+    <parent link="base_link"/>
+    <child link="gonecksx"/>
+    <origin xyz="${0.15-goshift_x} 0.09 ${-0.060+global_z_offset}" rpy="1.5708 0 0"/>
+  </joint>
+  <link name="goaneckshoulders">
+    <visual>
+      <geometry>
+        <cylinder radius="0.06" length="0.18"/>
+      </geometry>
+      <material name="gray">
+        <color rgba="${gray}"/>
+      </material>
+      <origin xyz="0 0 0" rpy="0 0 0"/>
+    </visual>
+  </link>
+  <joint name="goaneckshoulders_to_base" type="fixed">
+    <parent link="base_link"/>
+    <child link="goaneckshoulders"/>
+    <origin xyz="${0.15-goshift_x} 0 ${-0.060+global_z_offset}" rpy="1.5708 0 0"/>
+  </joint>
+  <link name="legsx">
+    <visual>
+      <geometry>
+        <box size="0.70 0.12 0.36"/>
       </geometry>
       <material name="orange">
@@ -244,14 +332,13 @@
     </visual>
   </link>
-  <joint name="goback_to_base" type="fixed">
-    <parent link="base_link"/>
-    <child link="goback"/>
-    <origin xyz="${(-gobody_length / 2) -goshift_x} 0 ${-gobody_fourth_of_y+global_z_offset}" rpy="${halfpi} 0 0"/>
-  </joint>
-  <!-- Back corners and neck-shoulder connector -->
-  <link name="gobackdx">
-    <visual>
-      <geometry>
-        <sphere radius="${gobody_fourth_of_y}"/>
+  <joint name="legsx_to_base" type="fixed">
+    <parent link="base_link"/>
+    <child link="legsx"/>
+    <origin xyz="${0-goshift_x} 0.1 ${-0.32+global_z_offset}" rpy="0 0 0"/>
+  </joint>
+  <link name="legdx">
+    <visual>
+      <geometry>
+        <box size="0.70 0.12 0.36"/>
       </geometry>
       <material name="orange">
@@ -261,105 +348,8 @@
     </visual>
   </link>
-  <joint name="gobackdx_to_base" type="fixed">
-    <parent link="base_link"/>
-    <child link="gobackdx"/>
-    <origin xyz="${(-gobody_length / 2) -goshift_x} ${-gobody_fourth_of_y *2} ${-gobody_fourth_of_y+global_z_offset}" rpy="${halfpi} 0 0"/>
-  </joint>
-  <link name="gobacksx">
-    <visual>
-      <geometry>
-        <sphere radius="${gobody_fourth_of_y}"/>
-      </geometry>
-      <material name="orange">
-        <color rgba="${orange}"/>
-      </material>
-      <origin xyz="0 0 0" rpy="0 0 0"/>
-    </visual>
-  </link>
-  <joint name="gobacksx_to_base" type="fixed">
-    <parent link="base_link"/>
-    <child link="gobacksx"/>
-    <origin xyz="${(-gobody_length / 2) -goshift_x} ${gobody_fourth_of_y * 2} ${-gobody_fourth_of_y+global_z_offset}" rpy="${halfpi} 0 0"/>
-  </joint>
-<link name="goneckdx">
-    <visual>
-      <geometry>
-        <sphere radius="${gobody_fourth_of_y}"/>
-      </geometry>
-      <material name="orange">
-        <color rgba="${orange}"/>
-      </material>
-      <origin xyz="0 0 0" rpy="0 0 0"/>
-    </visual>
-  </link>
-  <joint name="goneckdx_to_base" type="fixed">
-    <parent link="base_link"/>
-    <child link="goneckdx"/>
-    <origin xyz="${(gobody_length / 2) -goshift_x} ${-gobody_fourth_of_y * 2} ${-gobody_fourth_of_y+global_z_offset}" rpy="${halfpi} 0 0"/>
-  </joint>
-<link name="gonecksx">
-    <visual>
-      <geometry>
-        <sphere radius="${gobody_fourth_of_y}"/>
-      </geometry>
-      <material name="orange">
-        <color rgba="${orange}"/>
-      </material>
-      <origin xyz="0 0 0" rpy="0 0 0"/>
-    </visual>
-  </link>
-  <joint name="gonecksx_to_base" type="fixed">
-    <parent link="base_link"/>
-    <child link="gonecksx"/>
-    <origin xyz="${(gobody_length / 2) -goshift_x} ${gobody_fourth_of_y * 2} ${-gobody_fourth_of_y+global_z_offset}" rpy="${halfpi} 0 0"/>
-  </joint>
-  <link name="goaneckshoulders">
-    <visual>
-      <geometry>
-        <cylinder radius="${gobody_fourth_of_y}" length="${gobody_fourth_of_y * 4}"/>
-      </geometry>
-      <material name="orange">
-        <color rgba="${orange}"/>
-      </material>
-      <origin xyz="0 0 0" rpy="0 0 0"/>
-    </visual>
-  </link>
-  <joint name="goaneckshoulders_to_base" type="fixed">
-    <parent link="base_link"/>
-    <child link="goaneckshoulders"/>
-    <origin xyz="${(gobody_length / 2) -goshift_x} 0 ${-gobody_fourth_of_y+global_z_offset}" rpy="${halfpi} 0 0"/>
-  </joint>
-  <!-- Legs occupancy -->
-  <link name="legsx">
-    <visual>
-      <geometry>
-        <box size="0.70 ${gobody_fourth_of_y} ${0.2 + (gobody_fourth_of_y * 2)}"/>
-      </geometry>
-      <material name="orange">
-        <color rgba="${orange}"/>
-      </material>
-      <origin xyz="0 0 0" rpy="0 0 0"/>
-    </visual>
-  </link>
-  <joint name="legsx_to_base" type="fixed">
-    <parent link="base_link"/>
-    <child link="legsx"/>
-    <origin xyz="${-goshift_x} ${gobody_fourth_of_y * 5 / 2} ${-((0.2 + (gobody_fourth_of_y * 2)) / 2) - gobody_fourth_of_y + global_z_offset}" rpy="0 0 0"/>
-  </joint>
-  <link name="legdx">
-    <visual>
-      <geometry>
-        <box size="0.70 ${gobody_fourth_of_y} ${0.2 + (gobody_fourth_of_y * 2)}"/>
-      </geometry>
-      <material name="orange">
-        <color rgba="${orange}"/>
-      </material>
-      <origin xyz="0 0 0" rpy="0 0 0"/>
-    </visual>
-  </link>
   <joint name="legdx_to_base" type="fixed">
     <parent link="base_link"/>
     <child link="legdx"/>
-    <origin xyz="${-goshift_x} ${-gobody_fourth_of_y * 5 / 2} ${-((0.2 + (gobody_fourth_of_y * 2)) / 2) - gobody_fourth_of_y + global_z_offset}" rpy="0 0 0"/>
+    <origin xyz="${0-goshift_x} -0.1 ${-0.32+global_z_offset}" rpy="0 0 0"/>
   </joint>
 </robot>
