Commit message: Better structurization of launch files

File: helios16p_ws/install/helios16p_cane_robot/share/helios16p_cane_robot/urdf/helios16p.urdf.xacro (robot description, xacro)
@@ -36,5 +36,5 @@
   <xacro:property name="lidar_z" value="0.05"/>
   <!-- Base Link Its the "squared" part of the lidar base -->
-  <link name="base_link">
+  <link name="base_l">
     <visual>
       <geometry>
@@ -60,5 +60,5 @@
   </link>
   <joint name="base_round_to_base" type="fixed">
-    <parent link="base_link"/>
+    <parent link="base_l"/>
     <child link="base_round_part"/>
     <origin xyz="0 0 ${base_round_z+global_z_offset}" rpy="0 0 0"/>
@@ -77,5 +77,5 @@
   </link>
   <joint name="top_to_base" type="fixed">
-    <parent link="base_link"/>
+    <parent link="base_l"/>
     <child link="top_link"/>
     <origin xyz="0 0 ${top_z+global_z_offset}" rpy="0 0 0"/>
@@ -94,5 +94,5 @@
   </link>
   <joint name="top_round_to_base" type="fixed">
-    <parent link="base_link"/>
+    <parent link="base_l"/>
     <child link="top_round_part"/>
     <origin xyz="0 0 ${top_z+global_z_offset}" rpy="0 0 0"/>
@@ -111,5 +111,5 @@
   </link>
   <joint name="sx_pillar_to_base" type="fixed">
-    <parent link="base_link"/>
+    <parent link="base_l"/>
     <child link="sx_pillar"/>
     <origin xyz="-0.055 0.05 ${pillar_z+global_z_offset}" rpy="0 0 0"/>
@@ -128,5 +128,5 @@
   </link>
   <joint name="dx_pillar_to_base" type="fixed">
-    <parent link="base_link"/>
+    <parent link="base_l"/>
     <child link="dx_pillar"/>
     <origin xyz="-0.055 -0.05 ${pillar_z+global_z_offset}" rpy="0 0 0"/>
@@ -145,5 +145,5 @@
   </link>
   <joint name="base_to_lidar" type="fixed">
-    <parent link="base_link"/>
+    <parent link="base_l"/>
     <child link="lidar_link"/>
     <origin xyz="0 0 ${lidar_z+global_z_offset}" rpy="0 0 0"/>
@@ -162,5 +162,5 @@
   </link>
   <joint name="gobody_to_base" type="fixed">
-    <parent link="base_link"/>
+    <parent link="base_l"/>
     <child link="gobody"/>
     <origin xyz="${0-goshift_x} 0 ${-gobody_fourth_of_y+global_z_offset}" rpy="0 0 0"/>
@@ -178,5 +178,5 @@
   </link>
   <joint name="gobodysx_to_base" type="fixed">
-    <parent link="base_link"/>
+    <parent link="base_l"/>
     <child link="gobodysx"/>
     <origin xyz="${0-goshift_x} ${gobody_fourth_of_y} ${-gobody_fourth_of_y+global_z_offset}" rpy="0 ${halfpi} 0"/>
@@ -194,5 +194,5 @@
   </link>
   <joint name="gobodydx_to_base" type="fixed">
-    <parent link="base_link"/>
+    <parent link="base_l"/>
     <child link="gobodydx"/>
     <origin xyz="${0-goshift_x} ${-gobody_fourth_of_y} ${-gobody_fourth_of_y+global_z_offset}" rpy="0 ${halfpi} 0"/>
@@ -211,5 +211,5 @@
   </link>
   <joint name="goneck_to_base" type="fixed">
-    <parent link="base_link"/>
+    <parent link="base_l"/>
     <child link="goneck"/>
     <origin xyz="${(gobody_length / 2) + (gobody_fourth_of_y / 2) -goshift_x} 0 ${-gobody_fourth_of_y+global_z_offset}" rpy="0 0 0"/>
@@ -228,5 +228,5 @@
   </link>
   <joint name="gohead_to_base" type="fixed">
-    <parent link="base_link"/>
+    <parent link="base_l"/>
     <child link="gohead"/>
     <origin xyz="${(gobody_length / 2) + (gobody_fourth_of_y * 2) - goshift_x} 0 ${-gobody_fourth_of_y+global_z_offset}" rpy="${halfpi} 0 0"/>
@@ -245,5 +245,5 @@
   </link>
   <joint name="goback_to_base" type="fixed">
-    <parent link="base_link"/>
+    <parent link="base_l"/>
     <child link="goback"/>
     <origin xyz="${(-gobody_length / 2) -goshift_x} 0 ${-gobody_fourth_of_y+global_z_offset}" rpy="${halfpi} 0 0"/>
@@ -262,5 +262,5 @@
   </link>
   <joint name="gobackdx_to_base" type="fixed">
-    <parent link="base_link"/>
+    <parent link="base_l"/>
     <child link="gobackdx"/>
     <origin xyz="${(-gobody_length / 2) -goshift_x} ${-gobody_fourth_of_y *2} ${-gobody_fourth_of_y+global_z_offset}" rpy="${halfpi} 0 0"/>
@@ -278,5 +278,5 @@
   </link>
   <joint name="gobacksx_to_base" type="fixed">
-    <parent link="base_link"/>
+    <parent link="base_l"/>
     <child link="gobacksx"/>
     <origin xyz="${(-gobody_length / 2) -goshift_x} ${gobody_fourth_of_y * 2} ${-gobody_fourth_of_y+global_z_offset}" rpy="${halfpi} 0 0"/>
@@ -294,5 +294,5 @@
   </link>
   <joint name="goneckdx_to_base" type="fixed">
-    <parent link="base_link"/>
+    <parent link="base_l"/>
     <child link="goneckdx"/>
     <origin xyz="${(gobody_length / 2) -goshift_x} ${-gobody_fourth_of_y * 2} ${-gobody_fourth_of_y+global_z_offset}" rpy="${halfpi} 0 0"/>
@@ -310,5 +310,5 @@
   </link>
   <joint name="gonecksx_to_base" type="fixed">
-    <parent link="base_link"/>
+    <parent link="base_l"/>
     <child link="gonecksx"/>
     <origin xyz="${(gobody_length / 2) -goshift_x} ${gobody_fourth_of_y * 2} ${-gobody_fourth_of_y+global_z_offset}" rpy="${halfpi} 0 0"/>
@@ -326,5 +326,5 @@
   </link>
   <joint name="goaneckshoulders_to_base" type="fixed">
-    <parent link="base_link"/>
+    <parent link="base_l"/>
     <child link="goaneckshoulders"/>
     <origin xyz="${(gobody_length / 2) -goshift_x} 0 ${-gobody_fourth_of_y+global_z_offset}" rpy="${halfpi} 0 0"/>
@@ -343,5 +343,5 @@
   </link>
   <joint name="legsx_to_base" type="fixed">
-    <parent link="base_link"/>
+    <parent link="base_l"/>
     <child link="legsx"/>
     <origin xyz="${-goshift_x} ${gobody_fourth_of_y * 5 / 2} ${-((0.2 + (gobody_fourth_of_y * 2)) / 2) - gobody_fourth_of_y + global_z_offset}" rpy="0 0 0"/>
@@ -359,5 +359,5 @@
   </link>
   <joint name="legdx_to_base" type="fixed">
-    <parent link="base_link"/>
+    <parent link="base_l"/>
     <child link="legdx"/>
     <origin xyz="${-goshift_x} ${-gobody_fourth_of_y * 5 / 2} ${-((0.2 + (gobody_fourth_of_y * 2)) / 2) - gobody_fourth_of_y + global_z_offset}" rpy="0 0 0"/>
