Commit message: [Polished launch files structure]; [Included a launch file dedicated to benchmarking]; [Modified urdf xacro main link name from base to base_link]; [Included cloudini_ros package]: to minimize data transmission overhead thanks to cloudini compression of pointcloud rslidar_points].

File: helios16p_container_files/helios16p_ws/src/go1_description/xacro/helios16p_LiDAR.urdf.xacro (robot description, xacro)
@@ -33,5 +33,5 @@
 <xacro:macro name="lidar_macro" params="parent">
   <!-- Link principale - è la parte "squadrata" della base del lidar -->
-  <link name="${parent}_base_l">
+  <link name="${parent}_base_link">
     <visual>
       <geometry>
@@ -57,5 +57,5 @@
   </link>
   <joint name="${parent}_base_round_to_base" type="fixed">
-    <parent link="${parent}_base_l"/>
+    <parent link="${parent}_base_link"/>
     <child link="${parent}_base_round_part"/>
     <origin xyz="${global_x_lidar_shift} ${global_y_lidar_shift} ${global_z_lidar_shift + base_round_z}" rpy="0 0 0"/>
@@ -74,5 +74,5 @@
   </link>
   <joint name="${parent}_top_to_base" type="fixed">
-    <parent link="${parent}_base_l"/>
+    <parent link="${parent}_base_link"/>
     <child link="${parent}_top_link"/>
     <origin xyz="${global_x_lidar_shift} ${global_y_lidar_shift} ${global_z_lidar_shift + top_z}" rpy="0 0 0"/>
@@ -91,5 +91,5 @@
   </link>
   <joint name="${parent}_top_round_to_base" type="fixed">
-    <parent link="${parent}_base_l"/>
+    <parent link="${parent}_base_link"/>
     <child link="${parent}_top_round_part"/>
     <origin xyz="${global_x_lidar_shift} ${global_y_lidar_shift} ${global_z_lidar_shift + top_z}" rpy="0 0 0"/>
@@ -108,5 +108,5 @@
   </link>
   <joint name="${parent}_sx_pillar_to_base" type="fixed">
-    <parent link="${parent}_base_l"/>
+    <parent link="${parent}_base_link"/>
     <child link="${parent}_sx_pillar"/>
     <origin xyz="${global_x_lidar_shift - 0.055} ${global_y_lidar_shift + 0.05} ${global_z_lidar_shift + pillar_z}" rpy="0 0 0"/>
@@ -125,5 +125,5 @@
   </link>
   <joint name="${parent}_dx_pillar_to_base" type="fixed">
-    <parent link="${parent}_base_l"/>
+    <parent link="${parent}_base_link"/>
     <child link="${parent}_dx_pillar"/>
     <origin xyz="${global_x_lidar_shift - 0.055} ${global_y_lidar_shift - 0.05} ${global_z_lidar_shift + pillar_z}" rpy="0 0 0"/>
@@ -142,5 +142,5 @@
   </link>
   <joint name="${parent}_base_to_lidar" type="fixed">
-    <parent link="${parent}_base_l"/>
+    <parent link="${parent}_base_link"/>
     <child link="${parent}_lidar_link"/>
     <origin xyz="${global_x_lidar_shift} ${global_y_lidar_shift} ${global_z_lidar_shift + lidar_z}" rpy="0 0 0"/>

File: helios16p_container_files/helios16p_ws/src/go1_description/xacro/robot.xacro (robot description, xacro)
@@ -20,8 +20,8 @@
             <origin rpy="0 0 0" xyz="0 0 0"/>
             <parent link="world"/>
-            <child link="base"/>
+            <child link="base_link"/>
         </joint>
     </xacro:if>
-    <link name="base">
+    <link name="base_link">
         <visual>
             <origin rpy="0 0 0" xyz="0 0 0"/>
@@ -33,5 +33,5 @@
     <joint name="floating_base" type="fixed">
         <origin rpy="0 0 0" xyz="0 0 0"/>
-        <parent link="base"/>
+        <parent link="base_link"/>
         <child link="trunk"/>
     </joint>
@@ -128,7 +128,7 @@
     <!-- LiDAR mounted on the back of the robot -->
     <xacro:lidar_macro parent="trunk"/>
-    <joint name="trunk_to_lidar_base" type="fixed">
+    <joint name="trunk_to_lidar_base_link" type="fixed">
         <parent link="trunk"/>
-        <child link="trunk_base_l"/>
+        <child link="trunk_base_link"/>
         <origin xyz="0.05 0 0.05" rpy="0 0 0"/>
     </joint>
